Commit message: fixing sps and rtf

File: src/limo_description/urdf/limo_ackerman.xacro (robot description, xacro)
@@ -1,12 +1,23 @@
 <?xml version="1.0"?>
+<!--
+  LIMO Pro URDF for Gazebo Harmonic (v0.2 stable).
+  Changes vs original:
+    1. New xacro arg 'enable_camera' (default false). When false, the
+       RGBD camera macro is not instantiated at all and the camera
+       sensor is excluded from the URDF entirely. Pass enable_camera:=true
+       at xacro time for the perception-pipeline eval pass with
+       YOLOv8 + DeepSORT.
+    2. depth_camera frames are still emitted unconditionally so the TF
+       tree is stable regardless of camera state.
+-->
 <robot name="limo_ackerman" xmlns:xacro="http://ros.org/wiki/xacro">
   <!-- Arguments -->
   <xacro:arg name="robot_namespace" default="/" />
+  <xacro:arg name="use_gazebo" default="true" />
+  <xacro:arg name="enable_camera" default="false" />
   <!-- Includes -->
-  <!-- On garde gazebo si tu veux, mais on évite de passer des blocks origin aux macros -->
-   <xacro:arg name="use_gazebo" default="true" />
-<xacro:if value="$(arg use_gazebo)">
-  <xacro:include filename="$(find limo_description)/urdf/limo_gazebo.gazebo"/>
-</xacro:if>
+  <xacro:if value="$(arg use_gazebo)">
+    <xacro:include filename="$(find limo_description)/urdf/limo_gazebo.gazebo"/>
+  </xacro:if>
   <!-- Properties -->
   <xacro:property name="M_PI" value="3.14159"/>
@@ -32,10 +43,16 @@
       model_name="limo" />
   </xacro:if>
-<xacro:if value="$(arg use_gazebo)">
-  <xacro:gz_lidar frame_prefix="laser" model_name="limo"/>
-  <xacro:gz_rgbd_camera frame_prefix="depth_camera" model_name="limo"/>
-  <xacro:gz_imu frame_prefix="imu" model_name="limo"/>
-</xacro:if>
-  <!-- Base link DOIT être la racine physique (Gazebo) -->
+  <xacro:wheel_friction_surface link_name="front_left_wheel_link"/>
+  <xacro:wheel_friction_surface link_name="front_right_wheel_link"/>
+  <xacro:wheel_friction_surface link_name="rear_left_wheel_link"/>
+  <xacro:wheel_friction_surface link_name="rear_right_wheel_link"/>
+  <xacro:if value="$(arg use_gazebo)">
+    <xacro:gz_lidar frame_prefix="laser" model_name="limo"/>
+    <xacro:gz_imu frame_prefix="imu" model_name="limo"/>
+    <xacro:if value="$(arg enable_camera)">
+      <xacro:gz_rgbd_camera frame_prefix="depth_camera" model_name="limo"/>
+    </xacro:if>
+  </xacro:if>
+  <!-- Base link DOIT etre la racine physique (Gazebo) -->
   <link name="base_link">
     <visual>
@@ -62,36 +79,34 @@
     <parent link="base_link"/>
     <child link="base_footprint"/>
-    <!-- on met footprint au sol -->
     <origin xyz="0 0 -0.15" rpy="0 0 0"/>
   </joint>
-      <!-- Laser frame -->
-    <link name="laser_link"/>
-    <joint name="laser_joint" type="fixed">
-      <parent link="base_link"/>
-      <child link="laser_link"/>
-      <!-- Ajuste xyz selon ton placement réel -->
-      <origin xyz="0.10 0.0 0.12" rpy="0 0 0"/>
-    </joint>
-      <!-- IMU frame -->
-    <link name="imu_link"/>
-    <joint name="imu_joint" type="fixed">
-      <parent link="base_link"/>
-      <child link="imu_link"/>
-      <origin xyz="0.0 0.0 0.10" rpy="0 0 0"/>
-    </joint>
-      <!-- Depth camera frame -->
-    <link name="depth_camera_link"/>
-    <joint name="depth_camera_joint" type="fixed">
-      <parent link="base_link"/>
-      <child link="depth_camera_link"/>
-      <origin xyz="0.12 0.0 0.14" rpy="0 0 0"/>
-    </joint>
-    <!-- Optical frame (REP-103: X right, Y down, Z forward) -->
-    <link name="depth_camera_optical_frame"/>
-    <joint name="depth_camera_optical_joint" type="fixed">
-      <parent link="depth_camera_link"/>
-      <child link="depth_camera_optical_frame"/>
-      <origin xyz="0 0 0" rpy="-1.57079632679 0 -1.57079632679"/>
-    </joint>
+  <!-- Laser frame -->
+  <link name="laser_link"/>
+  <joint name="laser_joint" type="fixed">
+    <parent link="base_link"/>
+    <child link="laser_link"/>
+    <origin xyz="0.10 0.0 0.12" rpy="0 0 0"/>
+  </joint>
+  <!-- IMU frame -->
+  <link name="imu_link"/>
+  <joint name="imu_joint" type="fixed">
+    <parent link="base_link"/>
+    <child link="imu_link"/>
+    <origin xyz="0.0 0.0 0.10" rpy="0 0 0"/>
+  </joint>
+  <!-- Depth camera frame (kept unconditionally for TF stability) -->
+  <link name="depth_camera_link"/>
+  <joint name="depth_camera_joint" type="fixed">
+    <parent link="base_link"/>
+    <child link="depth_camera_link"/>
+    <origin xyz="0.12 0.0 0.14" rpy="0 0 0"/>
+  </joint>
+  <!-- Optical frame (REP-103: X right, Y down, Z forward) -->
+  <link name="depth_camera_optical_frame"/>
+  <joint name="depth_camera_optical_joint" type="fixed">
+    <parent link="depth_camera_link"/>
+    <child link="depth_camera_optical_frame"/>
+    <origin xyz="0 0 0" rpy="-1.57079632679 0 -1.57079632679"/>
+  </joint>
   <!-- FRONT LEFT wheel -->
   <link name="front_left_wheel_link">
@@ -129,5 +144,4 @@
     </inertial>
     <visual>
-      <!-- Flip pour que le mesh "parte" vers -Y côté droit -->
       <origin xyz="0 0 0" rpy="0 0 ${M_PI}"/>
       <geometry>
@@ -176,5 +190,5 @@
     <dynamics damping="0.2" friction="0.0"/>
   </joint>
-    <!-- Rear right wheel -->
+  <!-- Rear right wheel -->
   <link name="rear_right_wheel_link">
     <inertial>
